File: Projet ELEC/mux 6x1.kicad_sch (KiCad schematic)
At the start: 24 parts, among them Q1 ZXM61N02F, Q2 ZXM61N02F, Q3 ZXM61N02F, Q5 ZXM61N02F, Q6 ZXM61N02F, Q7 ZXM61N02F, U2 74LS21, U3 74LS21, U4 74LS21, U5 74LS21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

Commit message: chore: update project to latest version (what's the point of git)
* Projet ELEC/Projet ELEC.kicad_pcb
* Projet ELEC/Projet ELEC.kicad_sch
* Projet ELEC/demux 1x6.kicad_sch
* Projet ELEC/keyboard.kicad_sch
* Projet ELEC/mux 6x1.kicad_sch
* Projet ELEC/stm32.kicad_sch
Parts:
- removed U4: 74LS21, Package_DIP:DIP-14_W7.62mm, symbol 74xx:74LS21
Connections:
- net VCC is gone; now on net +3.3V: R11.1, R12.1, R13.1, R7.1, R8.1, R9.1
- net +5V renamed +3.3V
Changed lines of the file:
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@@
 	(paper "A4")
 	(junction
-		(at 87.63 181.61)
-		(diameter 0)
-		(color 0 0 0 0)
-	)
-	(junction
 		(at 102.87 85.09)
 		(diameter 0)
@@
 	)
 	(junction
-		(at 87.63 156.21)
-		(diameter 0)
-		(color 0 0 0 0)
-	)
-	(junction
 		(at 80.01 19.05)
 		(diameter 0)
@@
 	(wire
 		(pts
-			(xy 101.6 181.61) (xy 87.63 181.61)
+			(xy 73.66 181.61) (xy 101.6 181.61)
 		)
 		(stroke
@@
 	(wire
 		(pts
-			(xy 87.63 181.61) (xy 73.66 181.61)
-		)
-		(stroke
-			(width 0)
-			(type default)
-		)
-	)
-	(wire
-		(pts
 			(xy 157.48 156.21) (xy 143.51 156.21)
 		)
@@
 	(wire
 		(pts
-			(xy 101.6 156.21) (xy 87.63 156.21)
-		)
-		(stroke
-			(width 0)
-			(type default)
-		)
-	)
-	(wire
-		(pts
 			(xy 31.75 138.43) (xy 43.18 138.43)
 		)
@@
 	(wire
 		(pts
-			(xy 64.77 156.21) (xy 87.63 156.21)
+			(xy 64.77 156.21) (xy 101.6 156.21)
 		)
 		(stroke
@@
 			)
 		)
-		(property "Value" "VCC"
-			(at 177.8 113.03 0)
+		(property "Value" "+3.3V"
+			(at 179.07 113.0299 90)
 			(effects
 				(font
 					(size 1.27 1.27)
 				)
+				(justify left)
 			)
 		)
@@
 			)
 		)
-		(property "Value" "VCC"
+		(property "Value" "+3.3V"
 			(at 31.75 86.36 0)
 			(effects
@@
 			)
 		)
-		(property "Value" "VCC"
-			(at 139.7 113.03 0)
+		(property "Value" "+3.3V"
+			(at 140.97 113.0299 90)
 			(effects
 				(font
 					(size 1.27 1.27)
 				)
+				(justify left)
 			)
 		)
@@
 			)
 		)
-		(property "Value" "+5V"
-			(at 173.99 181.61 0)
+		(property "Value" "+3.3V"
+			(at 172.72 181.6099 90)
 			(effects
 				(font
 					(size 1.27 1.27)
 				)
+				(justify left)
 			)
 		)
@@
 			)
 		)
-		(property "Value" "VCC"
+		(property "Value" "+3.3V"
 			(at 31.75 121.92 0)
 			(effects
@@
 	)
 	(symbol
-		(lib_id "74xx:74LS21")
-		(at 87.63 168.91 180)
-		(unit 3)
-		(exclude_from_sim no)
-		(in_bom yes)
-		(on_board yes)
-		(dnp no)
-		(fields_autoplaced yes)
-		(property "Reference" "U4"
-			(at 81.28 170.1801 0)
-			(effects
-				(font
-					(size 1.27 1.27)
-				)
-				(justify left)
-			)
-		)
-		(property "Value" "74LS21"
-			(at 81.28 167.6401 0)
-			(effects
-				(font
-					(size 1.27 1.27)
-				)
-				(justify left)
-			)
-		)
-		(property "Footprint" "Package_DIP:DIP-14_W7.62mm"
-			(at 87.63 168.91 0)
-			(effects
-				(font
-					(size 1.27 1.27)
-				)
-				(hide yes)
-			)
-		)
-		(property "Datasheet" "http://www.ti.com/lit/gpn/sn74LS21"
-			(at 87.63 168.91 0)
-			(effects
-				(font
-					(size 1.27 1.27)
-				)
-				(hide yes)
-			)
-		)
-		(property "Description" "Dual 4-input AND"
-			(at 87.63 168.91 0)
-			(effects
-				(font
-					(size 1.27 1.27)
-				)
-				(hide yes)
-			)
-		)
-		(pin "10"
-		)
-		(pin "14"
-		)
-		(pin "9"
-		)
-		(pin "12"
-		)
-		(pin "6"
-		)
-		(pin "7"
-		)
-		(pin "8"
-		)
-		(pin "4"
-		)
-		(pin "1"
-		)
-		(pin "2"
-		)
-		(pin "13"
-		)
-		(pin "5"
-		)
-		(instances
-			(project "keybaord"
-				(path "/0ffb217f-e60b-4e29-93ea-87d2d0bc15d5"
-					(reference "U4")
-					(unit 3)
-				)
-			)
-			(project "Projet ELEC"
-				(path "/2d0c4a09-24e5-4892-bf2e-0a851a14e0ff/ce375f09-db8e-41ad-aaf2-7f45cfa7dab4"
-					(reference "U4")
-					(unit 3)
-				)
-			)
-		)
-	)
-	(symbol
 		(lib_id "Transistor_FET:ZXM61N02F")
 		(at 201.93 115.57 90)
@@
 			)
 		)
-		(property "Value" "VCC"
+		(property "Value" "+3.3V"
 			(at 31.75 48.26 0)
 			(effects
@@
 			)
 		)
-		(property "Value" "VCC"
-			(at 101.6 113.03 0)
+		(property "Value" "+3.3V"
+			(at 102.87 113.0299 90)
 			(effects
 				(font
 					(size 1.27 1.27)
 				)
+				(justify left)
 			)
 		)
