File: Projet ELEC/stm32.kicad_sch (KiCad schematic)
At the start: 20 parts, among them SW1 SW_Push, U8 STM32F103RBTx, U9 STM32F103C8Tx

Commit message: [*] stm32 decoupling caps
Parts:
- removed BZ1: Buzzer, Buzzer_Beeper:Buzzer_TDK_PS1240P02BT_D12.2mm_H6.5mm, symbol Device:Buzzer
- removed C1, C10, C2, C3, C4, C5, C6, C7, C8, C9: 10picoF, Capacitor_SMD:C_0201_0603Metric, symbol Device:C
- removed SW1: SW_Push, Button_Switch_SMD:SW_Push_1P1T_NO_CK_PTS125Sx43PSMTR, symbol Switch:SW_Push
- removed U8: STM32F103RBTx, Package_QFP:LQFP-64_10x10mm_P0.5mm, symbol MCU_ST_STM32F1:STM32F103RBTx
- added C11, C12, C13, C14, C17: 100nF, Capacitor_SMD:C_0201_0603Metric, symbol Device:C
- added C15: 10uF, Capacitor_SMD:C_0201_0603Metric, symbol Device:C
- added C16: 1uF, Capacitor_SMD:C_0201_0603Metric, symbol Device:C
- U9: value STM32F103C8Tx -> STM32F103C8T6
Connections:
- net GND: now also U9.44 (BOOT0), C11.2, C12.2, C13.2, C14.2, C15.2, C16.2, C17.2
- net at 3v3.MP (MountPin), U9.1 (VBAT), U9.24 (VDD)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: now also C11.1, C12.1, C13.1, C14.1, C15.1, C16.1, C17.1
- net BOOT1: now reaches U9.20 (PB2)
Other:
- note removed: "DEMUX 6x1 ROW selection"
- note removed: "MUX 1x6 COL selection"
- moved on the sheet: 3v3, NRST
