File: Projet ELEC/Projet ELEC.kicad_pcb (KiCad board)
At the start: 2 copper layers, 112 parts, among them Q1 ZXM61N02F, Q2 ZXM61N02F, Q3 ZXM61N02F, Q5 ZXM61N02F, Q6 ZXM61N02F, Q7 ZXM61N02F, SW1 SW_TOUCHE, SW10 SW_TOUCHE, SW11 SW_TOUCHE, SW12 SW_TOUCHE, SW13 SW_TOUCHE, SW14 SW_TOUCHE, SW15 SW_TOUCHE, SW16 SW_TOUCHE, SW17 SW_TOUCHE, SW18 SW_TOUCHE, SW19 SW_TOUCHE, SW2 SW_TOUCHE, SW20 SW_TOUCHE, SW21 SW_TOUCHE, SW22 SW_TOUCHE, SW23 SW_TOUCHE, SW24 SW_TOUCHE, SW25 SW_TOUCHE, SW26 SW_TOUCHE, SW27 SW_TOUCHE, SW28 SW_TOUCHE, SW29 SW_TOUCHE, SW3 SW_TOUCHE, SW30 SW_TOUCHE, SW31 SW_TOUCHE, SW32 SW_TOUCHE, SW33 SW_TOUCHE, SW34 SW_TOUCHE, SW35 SW_TOUCHE, SW36 SW_TOUCHE, SW4 SW_TOUCHE, SW5 SW_TOUCHE, SW6 SW_TOUCHE, SW7 SW_TOUCHE, SW8 SW_TOUCHE, SW9 SW_TOUCHE, U2 74LS21, U2-demux1 74LS21, U3 74LS21, U3-demux1 74LS21, U4 74LS21, U4-demux1 74LS21, U5 74LS21, U6 4071, U7 4071, U8 STM32F103RBTx

Commit message: fix ta merde quentin
Routing:
- net (no net): track 103.2 -> 387.7 mm
Changed lines of the file:
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@@
+	)
+	(segment
+		(start 33.25 -5.25)
+		(end -24.25 -5.25)
+		(width 0.2)
+		(layer "B.Cu")
+		(net 0)
+	)
+	(segment
+		(start -21 -11)
+		(end -21.5 -11)
+		(width 0.2)
+		(layer "B.Cu")
+		(net 0)
 	)
 	(segment
@@
 	)
 	(segment
+		(start -34 4.5)
+		(end -35 4.5)
+		(width 0.2)
+		(layer "B.Cu")
+		(net 0)
+	)
+	(segment
+		(start -21.5 -11)
+		(end -25.5 -11)
+		(width 0.2)
+		(layer "B.Cu")
+		(net 0)
+	)
+	(segment
+		(start -35 4.5)
+		(end -35.5 4)
+		(width 0.2)
+		(layer "B.Cu")
+		(net 0)
+	)
+	(segment
+		(start -28.5 -23)
+		(end -28.5 -14.5)
+		(width 0.2)
+		(layer "B.Cu")
+		(net 0)
+	)
+	(segment
 		(start 9.5 61)
 		(end 9.5 76)
@@
 	)
 	(segment
+		(start -24.25 -5.25)
+		(end -34 4.5)
+		(width 0.2)
+		(layer "B.Cu")
+		(net 0)
+	)
+	(segment
 		(start 10 91.5)
 		(end 14 91.5)
@@
 	)
 	(segment
-		(start 9.5 16.5)
-		(end 9.5 31)
-		(width 0.2)
-		(layer "B.Cu")
-		(net 0)
-	)
-	(segment
-		(start 9.5 16)
-		(end 9.5 16.5)
+		(start 34 -23)
+		(end 42.5 -14.5)
+		(width 0.2)
+		(layer "B.Cu")
+		(net 0)
+	)
+	(segment
+		(start -28.5 -38.5)
+		(end -28.5 -23)
+		(width 0.2)
+		(layer "B.Cu")
+		(net 0)
+	)
+	(segment
+		(start -35.5 4)
+		(end -46.5 4)
 		(width 0.2)
 		(layer "B.Cu")
@@
 	)
 	(segment
+		(start -43 -21)
+		(end -42.5 -21.5)
+		(width 0.2)
+		(layer "B.Cu")
+		(net 0)
+	)
+	(segment
+		(start -46.5 -0.5)
+		(end -52 -6)
+		(width 0.2)
+		(layer "B.Cu")
+		(net 0)
+	)
+	(segment
 		(start 9.5 45.5)
 		(end 10.5 46.5)
@@
 	)
 	(segment
+		(start -42.5 -21.5)
+		(end -42.5 -28.5)
+		(width 0.2)
+		(layer "B.Cu")
+		(net 0)
+	)
+	(segment
 		(start 9.5 13.5)
 		(end 9.5 16)
@@
 	)
 	(segment
+		(start -46.5 4)
+		(end -46.5 -0.5)
+		(width 0.2)
+		(layer "B.Cu")
+		(net 0)
+	)
+	(segment
+		(start -40 -16.5)
+		(end -39.5 -16)
+		(width 0.2)
+		(layer "B.Cu")
+		(net 0)
+	)
+	(segment
 		(start 9.5 76)
 		(end 9.5 91)
@@
 	)
 	(segment
+		(start -28.5 -14.5)
+		(end -29 -14.5)
+		(width 0.2)
+		(layer "B.Cu")
+		(net 0)
+	)
+	(segment
+		(start -42.5 -28.5)
+		(end -30.5 -40.5)
+		(width 0.2)
+		(layer "B.Cu")
+		(net 0)
+	)
+	(segment
+		(start -28.5 -23)
+		(end 34 -23)
+		(width 0.2)
+		(layer "B.Cu")
+		(net 0)
+	)
+	(segment
+		(start 42.5 -14.5)
+		(end 33.25 -5.25)
+		(width 0.2)
+		(layer "B.Cu")
+		(net 0)
+	)
+	(segment
 		(start 10 76.5)
 		(end 13.5 76.5)
@@
 	)
 	(segment
+		(start -52 -6)
+		(end -52 -7)
+		(width 0.2)
+		(layer "B.Cu")
+		(net 0)
+	)
+	(segment
+		(start -25.5 -11)
+		(end -29 -14.5)
+		(width 0.2)
+		(layer "B.Cu")
+		(net 0)
+	)
+	(segment
 		(start 10.5 46.5)
 		(end 13.5 46.5)
@@
 	)
 	(segment
+		(start -52 -7)
+		(end -42.5 -16.5)
+		(width 0.2)
+		(layer "B.Cu")
+		(net 0)
+	)
+	(segment
+		(start 9.5 16)
+		(end 9.5 31)
+		(width 0.2)
+		(layer "B.Cu")
+		(net 0)
+	)
+	(segment
+		(start -39.5 -14.5)
+		(end -43 -18)
+		(width 0.2)
+		(layer "B.Cu")
+		(net 0)
+	)
+	(segment
+		(start -21.5 -8)
+		(end -24.25 -5.25)
+		(width 0.2)
+		(layer "B.Cu")
+		(net 0)
+	)
+	(segment
 		(start 10 31.5)
 		(end 13.5 31.5)
@@
 	)
 	(segment
+		(start -21.5 -11)
+		(end -21.5 -8)
+		(width 0.2)
+		(layer "B.Cu")
+		(net 0)
+	)
+	(segment
 		(start 9.5 31)
 		(end 10 31.5)
@@
 	)
 	(segment
-		(start 9.5 16.5)
-		(end 13.5 16.5)
+		(start -39 -16)
+		(end -37.5 -14.5)
+		(width 0.2)
+		(layer "B.Cu")
+		(net 0)
+	)
+	(segment
+		(start -30.5 -40.5)
+		(end -28.5 -38.5)
+		(width 0.2)
+		(layer "B.Cu")
+		(net 0)
+	)
+	(segment
+		(start -37 -14.5)
+		(end -39.5 -14.5)
+		(width 0.2)
+		(layer "B.Cu")
+		(net 0)
+	)
+	(segment
+		(start -39.5 -16)
+		(end -39 -16)
+		(width 0.2)
+		(layer "B.Cu")
+		(net 0)
+	)
+	(segment
+		(start -42.5 -16.5)
+		(end -40 -16.5)
+		(width 0.2)
+		(layer "B.Cu")
+		(net 0)
+	)
+	(segment
+		(start -37.5 -14.5)
+		(end -37 -14.5)
 		(width 0.2)
 		(layer "B.Cu")
@@
 		(width 0.2)
 		(layer "B.Cu")
+		(net 0)
+	)
+	(segment
+		(start -29 -14.5)
+		(end -37 -14.5)
+		(width 0.2)
+		(layer "B.Cu")

Commit message: pcb updated
Parts:
- moved U4 180.7 mm to (137.2, -77.1)
- moved U3 16.1 mm to (-42.8, 66.1)
- moved U2 8.98 mm to (-42.8, 43.6)
- moved U5 8.03 mm to (-42.8, 21.1)
- moved U7 7.18 mm to (-86.8, 43.6)
- moved U6 6.41 mm to (-64.6, 43.6)
Routing:
- net (no net): track 387.7 -> 0.00 mm
- net GND: track 0.00 -> 79.1 mm
- net Row4: track 87.5 -> 159.7 mm
- net Row5: track 88.0 -> 151.7 mm
- net Row1: track 88.0 -> 148.1 mm
- net Row6: track 88.0 -> 145.6 mm
- net Row3: track 88.0 -> 139.7 mm
- net Row2: track 88.0 -> 138.8 mm
Other:
- board text added: "+3.3V"

Commit message: 6x1 almost done, just need to connect VCC/GND
Parts:
- moved U8 316.9 mm to (-11.2, -49.4)
- moved R13 187.4 mm to (-52.1, -14.5), turned to 0 degrees
- moved R12 186.9 mm to (-42.0, -14.5), turned to 0 degrees
- moved R11 186.7 mm to (-31.5, -14.5), turned to 0 degrees
- moved Q7 186.0 mm to (-47.0, -22.5)
- moved Q6 184.9 mm to (-37.0, -22.0)
- moved Q5 183.7 mm to (-26.5, -22.5)
- moved U7 63.5 mm to (-38.9, 85.2), turned to -90 degrees
- moved U6 44.1 mm to (-27.5, 67.4), turned to -90 degrees
- moved U3 44.1 mm to (-1.60, 81.6), turned to -90 degrees
- moved U2 42.0 mm to (-1.64, 51.8), turned to -90 degrees
- moved U5 41.2 mm to (-1.60, 21.6), turned to -90 degrees
Connections:
- Q5 pad 2: unconnected-(Q5-S-Pad2) -> GND
- Q6 pad 2: unconnected-(Q6-S-Pad2) -> GND
- Q7 pad 2: unconnected-(Q7-S-Pad2) -> GND
- U2 pad 1: Row4 -> Row3
- U2 pad 13: Net-(Q7-D) -> A0
- U2 pad 5: A0 -> Net-(Q7-D)
- U2 pad 9: Row3 -> Row4
- U6 pad 5: Net-(U2-Pad8) -> Net-(U2-Pad6)
- U6 pad 6: Net-(U2-Pad6) -> Net-(U2-Pad8)
Routing:
- net A0: track 0.00 -> 173.9 mm, vias 0 -> 6
- net Net-(Q6-D): track 0.00 -> 146.1 mm, vias 0 -> 2
- net A1: track 0.00 -> 124.3 mm, vias 0 -> 6
- net Net-(Q7-D): track 0.00 -> 123.8 mm
- net Net-(Q5-D): track 0.00 -> 99.7 mm, vias 0 -> 1
- net Net-(U5-Pad6): track 0.00 -> 51.2 mm, vias 0 -> 2
- net Row5: track 151.7 -> 104.1 mm
- net Net-(U5-Pad8): track 0.00 -> 47.2 mm, vias 0 -> 2
- net Row1: track 148.1 -> 104.1 mm
- net Row4: track 159.7 -> 119.3 mm
- net Net-(U3-Pad8): track 0.00 -> 37.9 mm
- net A2: track 0.00 -> 36.1 mm
- net Row3: track 139.7 -> 105.6 mm
- net Net-(U2-Pad6): track 0.00 -> 34.0 mm
- net Net-(U3-Pad6): track 0.00 -> 31.1 mm
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Other:
- board text removed: "+3.3V"

Commit message: 6x1 PCB done, saved this time
Routing:
- net GND: track 79.1 -> 277.3 mm, vias 0 -> 3
- net A2: track 36.1 -> 216.2 mm, vias 0 -> 2
- net DEMUX_OUTPUT: track 0.00 -> 159.3 mm, vias 0 -> 2
- net +5V: track 22.5 -> 126.9 mm, vias 0 -> 5

Commit message: PCB done, except ST, pin headers and a few resistors not connected to ground
Parts:
- removed U4: 74LS21, Package_DIP:DIP-14_W7.62mm
- moved BZ1 296.6 mm to (9.50, -95.6)
- moved C1 296.6 mm to (-10.9, -106.7)
- moved C10 296.6 mm to (-3.95, -109.1)
- moved C2 296.6 mm to (-9.20, -106.7)
- moved C3 296.6 mm to (-7.45, -106.7)
- moved C4 296.6 mm to (-5.70, -106.7)
- moved C5 296.6 mm to (-3.95, -106.7)
- moved C6 296.6 mm to (-10.9, -109.1)
- moved C7 296.6 mm to (-9.20, -109.1)
- moved C8 296.6 mm to (-7.45, -109.1)
- moved C9 296.6 mm to (-5.70, -109.1)
- moved reset_btn1 296.6 mm to (4.65, -107.0)
- moved R9 108.4 mm to (40.5, -37.4)
- moved Q3 96.7 mm to (36.0, -41.6)
- moved R8 92.9 mm to (55.0, -37.5)
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Routing:
- net +5V: track 126.9 -> 317.8 mm, vias 5 -> 7
- net NOT1_IN: track 0.00 -> 189.2 mm, vias 0 -> 6
- net NOT2_IN: track 0.00 -> 147.1 mm, vias 0 -> 2
- net NOT2_OUT: track 0.00 -> 128.8 mm, vias 0 -> 2
- net NOT1_OUT: track 0.00 -> 118.2 mm, vias 0 -> 1
- net NOT3_IN: track 0.00 -> 106.2 mm, vias 0 -> 2
- net NOT3_OUT: track 0.00 -> 96.0 mm, vias 0 -> 2
- net VCC: track 0.00 -> 66.1 mm
- net Net-(U2-demux1C-GND): track 0.00 -> 61.8 mm
- net GND: track 277.3 -> 319.8 mm, vias 3 -> 6
- net Col5: track 91.5 -> 106.8 mm
- net Col1: track 91.5 -> 106.8 mm
- net Col3: track 91.5 -> 106.8 mm
- net Col6: track 91.5 -> 104.6 mm
- net Col4: track 91.5 -> 104.6 mm
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
Commit message: fixed some switches not connected
Routing:
- net Net-(D4-K): track 0.00 -> 12.0 mm
- net Net-(D9-K): track 5.50 -> 12.0 mm
- net Net-(D8-K): track 5.52 -> 12.0 mm
- net Net-(D7-K): track 5.50 -> 12.0 mm
- net Net-(D6-K): track 5.52 -> 12.0 mm
- net Net-(D5-K): track 5.50 -> 12.0 mm
- net Net-(D36-K): track 5.50 -> 12.0 mm
- net Net-(D35-K): track 5.50 -> 12.0 mm
- net Net-(D34-K): track 5.50 -> 12.0 mm
- net Net-(D33-K): track 5.50 -> 12.0 mm
- net Net-(D32-K): track 5.50 -> 12.0 mm
- net Net-(D31-K): track 5.52 -> 12.0 mm
- net Net-(D30-K): track 5.52 -> 12.0 mm
- net Net-(D3-K): track 5.52 -> 12.0 mm
- net Net-(D29-K): track 5.52 -> 12.0 mm
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
Commit message: chore: update project to latest version (what's the point of git)
* Projet ELEC/Projet ELEC.kicad_pcb
* Projet ELEC/Projet ELEC.kicad_sch
* Projet ELEC/demux 1x6.kicad_sch
* Projet ELEC/keyboard.kicad_sch
* Projet ELEC/mux 6x1.kicad_sch
* Projet ELEC/stm32.kicad_sch
Parts:
- removed BZ1: Buzzer, Buzzer_Beeper:Buzzer_TDK_PS1240P02BT_D12.2mm_H6.5mm
- removed C1, C10, C2, C3, C4, C5, C6, C7, C8, C9: 10picoF, Capacitor_SMD:C_0201_0603Metric
- removed reset_btn1: SW_Push, Button_Switch_THT:SW_PUSH_6mm
- added 3v1: Conn_01x01_MountingPin, Connector_PinHeader_1.00mm:PinHeader_1x01_P1.00mm_Vertical, F.Cu at (99.3, 19.1)
- added BZ2: Buzzer, Buzzer_Beeper:Buzzer_TDK_PS1240P02BT_D12.2mm_H6.5mm, F.Cu at (81.5, -18.5)
- added GND1: Conn_01x01_MountingPin, Connector_PinHeader_1.00mm:PinHeader_1x01_P1.00mm_Vertical, F.Cu at (99.3, 14.5)
- added NRST1: Conn_01x01_MountingPin, Connector_PinHeader_1.00mm:PinHeader_1x01_P1.00mm_Vertical, F.Cu at (44.7, 7.10)
- added SWCLK1: Conn_01x01_MountingPin, Connector_PinHeader_1.00mm:PinHeader_1x01_P1.00mm_Vertical, F.Cu at (63.7, -2.70)
- added SWDIO1: Conn_01x01_MountingPin, Connector_PinHeader_1.00mm:PinHeader_1x01_P1.00mm_Vertical, F.Cu at (80.3, 4.30)
- SW1: value SW_TOUCHE -> SWR1C1
- SW10: renamed from SW25; value SW_TOUCHE -> SWR5C1
- SW11: renamed from SW31; value SW_TOUCHE -> SWR6C1
- SW12: renamed from SW8; value SW_TOUCHE -> SWR2C2
- SW13: renamed from SW14; value SW_TOUCHE -> SWR3C2
- SW14: renamed from SW20; value SW_TOUCHE -> SWR4C2
- SW15: renamed from SW26; value SW_TOUCHE -> SWR5C2
- SW16: renamed from SW32; value SW_TOUCHE -> SWR6C2
- SW17: renamed from SW9; value SW_TOUCHE -> SWR2C3
- SW18: renamed from SW15; value SW_TOUCHE -> SWR3C3
- SW19: renamed from SW21; value SW_TOUCHE -> SWR4C3
- SW2: value SW_TOUCHE -> SWR1C2
- SW20: renamed from SW27; value SW_TOUCHE -> SWR5C3
- SW21: renamed from SW33; value SW_TOUCHE -> SWR6C3
- SW22: renamed from SW10; value SW_TOUCHE -> SWR2C4
- SW23: renamed from SW16; value SW_TOUCHE -> SWR3C4
- SW24: renamed from SW22; value SW_TOUCHE -> SWR4C4
- SW25: renamed from SW28; value SW_TOUCHE -> SWR5C4
- SW26: renamed from SW34; value SW_TOUCHE -> SWR6C4
- SW27: renamed from SW11; value SW_TOUCHE -> SWR2C5
- SW28: renamed from SW17; value SW_TOUCHE -> SWR3C5
- SW29: renamed from SW23; value SW_TOUCHE -> SWR4C5
- SW3: value SW_TOUCHE -> SWR1C3
- SW30: renamed from SW29; value SW_TOUCHE -> SWR5C5
- SW31: renamed from SW35; value SW_TOUCHE -> SWR6C5
- SW32: renamed from SW12; value SW_TOUCHE -> SWR2C6
- SW33: renamed from SW18; value SW_TOUCHE -> SWR3C6
- SW34: renamed from SW24; value SW_TOUCHE -> SWR4C6
- SW35: renamed from SW30; value SW_TOUCHE -> SWR5C6
- SW36: value SW_TOUCHE -> SWR6C6
- SW4: value SW_TOUCHE -> SWR1C4
- SW5: value SW_TOUCHE -> SWR1C5
- SW6: value SW_TOUCHE -> SWR1C6
- SW7: value SW_TOUCHE -> SWR2C1
- SW8: renamed from SW13; value SW_TOUCHE -> SWR3C1
- SW9: renamed from SW19; value SW_TOUCHE -> SWR4C1
- U8: value STM32F103RBTx -> STM32F103C8Tx; footprint Package_QFP:LQFP-64_10x10mm_P0.5mm -> Package_QFP:LQFP-48_7x7mm_P0.5mm
- moved Q2 96.9 mm to (129.2, 15.6)
- moved DR1C1 96.9 mm to (106.4, 88.4)
- moved DR1C2 96.9 mm to (121.5, 88.4)
- moved DR1C3 96.9 mm to (136.4, 88.4)
- moved DR1C4 96.9 mm to (151.4, 88.4)
- moved DR1C5 96.9 mm to (166.4, 88.4)
- moved DR1C6 96.9 mm to (181.5, 88.4)
- moved DR2C1 96.9 mm to (106.4, 103.4)
- moved DR2C2 96.9 mm to (121.4, 103.4)
- moved DR2C3 96.9 mm to (136.5, 103.4)
- moved DR2C4 96.9 mm to (151.5, 103.4)
- moved DR2C5 96.9 mm to (166.4, 103.4)
- moved DR2C6 96.9 mm to (181.5, 103.4)
- moved DR3C1 96.9 mm to (106.4, 118.4)
- moved DR3C2 96.9 mm to (121.5, 118.4)
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- renumbered D6 to DR1C1, D5 to DR1C2, D4 to DR1C3, D3 to DR1C4, D2 to DR1C5, D1 to DR1C6, D12 to DR2C1, D11 to DR2C2, D10 to DR2C3, D9 to DR2C4, D8 to DR2C5, D7 to DR2C6, D23 to DR3C1, D21 to DR3C2, D19 to DR3C3, D17 to DR3C4, D15 to DR3C5, D13 to DR3C6, D24 to DR4C1, D22 to DR4C2, D20 to DR4C3, D18 to DR4C4, D16 to DR4C5, D14 to DR4C6, D30 to DR5C1, D29 to DR5C2, D28 to DR5C3, D27 to DR5C4, D26 to DR5C5, D25 to DR5C6, D31 to DR6C1, D36 to DR6C2, D35 to DR6C3, D34 to DR6C4, D33 to DR6C5, D32 to DR6C6
Connections:
- R11 pad 1: VCC -> +3.3V
- R12 pad 1: VCC -> +3.3V
- R13 pad 1: VCC -> +3.3V
- R7 pad 1: VCC -> +3.3V
- R8 pad 1: VCC -> +3.3V
- R9 pad 1: VCC -> +3.3V
- U2 pad 14: +5V -> +3.3V
- U2-demux1 pad 1: +5V -> +3.3V
- U2-demux1 pad 14: +5V -> +3.3V
- U2-demux1 pad 7: Net-(U2-demux1C-GND) -> GND
- U2-demux1 pad 9: +5V -> +3.3V
- U3 pad 14: +5V -> +3.3V
- U3-demux1 pad 1: +5V -> +3.3V
- U3-demux1 pad 14: +5V -> +3.3V
- U3-demux1 pad 7: Net-(U2-demux1C-GND) -> GND
- U3-demux1 pad 9: +5V -> +3.3V
- U4-demux1 pad 1: +5V -> +3.3V
- U4-demux1 pad 14: +5V -> +3.3V
- U4-demux1 pad 7: Net-(U2-demux1C-GND) -> GND
- U4-demux1 pad 9: +5V -> +3.3V
- U5 pad 14: +5V -> +3.3V
- U6 pad 14: +5V -> +3.3V
- U7 pad 14: +5V -> +3.3V
- U7 pad 4: DEMUX_OUTPUT -> MUX_OUTPUT
- U8 pad 10: NOT2_IN -> Net-(BZ2-+)
- U8 pad 11: NOT3_IN -> unconnected-(U8-PA1-Pad11)
- U8 pad 12: GND -> MUX_OUTPUT
- U8 pad 13: +3.3V -> unconnected-(U8-PA3-Pad13)
- U8 pad 18: GND -> unconnected-(U8-PB0-Pad18)
- U8 pad 19: +3.3V -> unconnected-(U8-PB1-Pad19)
- U8 pad 20: A2 -> unconnected-(U8-PB2-Pad20)
- U8 pad 21: DEMUX_OUTPUT -> SDA
- U8 pad 22: SWD0 -> SCL
- U8 pad 23: Net-(BZ1-+) -> GND
- U8 pad 24: unconnected-(U8-PC4-Pad24) -> +3.3V
- U8 pad 29: unconnected-(U8-PB10-Pad29) -> A2
- U8 pad 31: GND -> NOT1_IN
- U8 pad 32: +3.3V -> NOT2_IN
- U8 pad 33: unconnected-(U8-PB12-Pad33) -> NOT3_IN
- U8 pad 34: unconnected-(U8-PB13-Pad34) -> Net-(SWDIO1-Pin_1)
- U8 pad 35: unconnected-(U8-PB14-Pad35) -> GND
- U8 pad 36: unconnected-(U8-PB15-Pad36) -> +3.3V
- U8 pad 37: unconnected-(U8-PC6-Pad37) -> Net-(SWCLK1-Pin_1)
- U8 pad 44: unconnected-(U8-PA11-Pad44) -> GND
- U8 pad 46: SDA -> unconnected-(U8-PB9-Pad46)
- U8 pad 8: unconnected-(U8-PC0-Pad8) -> GND
- U8 pad 9: NOT1_IN -> +3.3V
Routing:
- net +3.3V: track 0.00 -> 689.4 mm, vias 0 -> 22
- net +5V: track 317.8 -> 0.00 mm, vias 7 -> 0
- net GND: track 319.8 -> 625.3 mm, vias 6 -> 11
- net MUX_OUTPUT: track 0.00 -> 174.5 mm, vias 0 -> 4
- net DEMUX_OUTPUT: track 159.3 -> 0.00 mm, vias 2 -> 0
- net VCC: track 66.1 -> 0.00 mm
- net Net-(BZ2-+): track 0.00 -> 62.1 mm
- net Net-(U2-demux1C-GND): track 61.8 -> 0.00 mm
- net Net-(SWDIO1-Pin_1): track 0.00 -> 18.6 mm, vias 0 -> 1
- net Net-(NRST1-Pin_1): track 0.00 -> 12.2 mm
- net A2: track 216.2 -> 223.7 mm
- net Net-(SWCLK1-Pin_1): track 0.00 -> 4.84 mm
- net A1: track 124.3 -> 128.4 mm
- net NOT1_IN: track 189.2 -> 186.5 mm
- net Row3: track 105.6 -> 104.2 mm
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Other:
- board outline added: 177.6 x 199.6 mm
