File: Projet ELEC/keyboard.kicad_sch (KiCad schematic)
At the start: 72 parts, among them SW1 SW_TOUCHE, SW10 SW_TOUCHE, SW11 SW_TOUCHE, SW12 SW_TOUCHE, SW13 SW_TOUCHE, SW14 SW_TOUCHE, SW15 SW_TOUCHE, SW16 SW_TOUCHE, SW17 SW_TOUCHE, SW18 SW_TOUCHE, SW19 SW_TOUCHE, SW2 SW_TOUCHE, SW20 SW_TOUCHE, SW21 SW_TOUCHE, SW22 SW_TOUCHE, SW23 SW_TOUCHE, SW24 SW_TOUCHE, SW25 SW_TOUCHE, SW26 SW_TOUCHE, SW27 SW_TOUCHE, SW28 SW_TOUCHE, SW29 SW_TOUCHE, SW3 SW_TOUCHE, SW30 SW_TOUCHE, SW31 SW_TOUCHE, SW32 SW_TOUCHE, SW33 SW_TOUCHE, SW34 SW_TOUCHE, SW35 SW_TOUCHE, SW36 SW_TOUCHE, SW4 SW_TOUCHE, SW5 SW_TOUCHE, SW6 SW_TOUCHE, SW7 SW_TOUCHE, SW8 SW_TOUCHE, SW9 SW_TOUCHE

Commit message: chore: update project to latest version (what's the point of git)
* Projet ELEC/Projet ELEC.kicad_pcb
* Projet ELEC/Projet ELEC.kicad_sch
* Projet ELEC/demux 1x6.kicad_sch
* Projet ELEC/keyboard.kicad_sch
* Projet ELEC/mux 6x1.kicad_sch
* Projet ELEC/stm32.kicad_sch
Parts:
- SW1: value SW_TOUCHE -> SWR1C1
- SW10: value SW_TOUCHE -> SWR2C4
- SW11: value SW_TOUCHE -> SWR2C5
- SW12: value SW_TOUCHE -> SWR2C6
- SW13: value SW_TOUCHE -> SWR3C1
- SW14: value SW_TOUCHE -> SWR3C2
- SW15: value SW_TOUCHE -> SWR3C3
- SW16: value SW_TOUCHE -> SWR3C4
- SW17: value SW_TOUCHE -> SWR3C5
- SW18: value SW_TOUCHE -> SWR3C6
- SW19: value SW_TOUCHE -> SWR4C1
- SW2: value SW_TOUCHE -> SWR1C2
- SW20: value SW_TOUCHE -> SWR4C2
- SW21: value SW_TOUCHE -> SWR4C3
- SW22: value SW_TOUCHE -> SWR4C4
- SW23: value SW_TOUCHE -> SWR4C5
- SW24: value SW_TOUCHE -> SWR4C6
- SW25: value SW_TOUCHE -> SWR5C1
- SW26: value SW_TOUCHE -> SWR5C2
- SW27: value SW_TOUCHE -> SWR5C3
- SW28: value SW_TOUCHE -> SWR5C4
- SW29: value SW_TOUCHE -> SWR5C5
- SW3: value SW_TOUCHE -> SWR1C3
- SW30: value SW_TOUCHE -> SWR5C6
- SW31: value SW_TOUCHE -> SWR6C1
- SW32: value SW_TOUCHE -> SWR6C2
- SW33: value SW_TOUCHE -> SWR6C3
- SW34: value SW_TOUCHE -> SWR6C4
- SW35: value SW_TOUCHE -> SWR6C5
- SW36: value SW_TOUCHE -> SWR6C6
- SW4: value SW_TOUCHE -> SWR1C4
- SW5: value SW_TOUCHE -> SWR1C5
- SW6: value SW_TOUCHE -> SWR1C6
- SW7: value SW_TOUCHE -> SWR2C1
- SW8: value SW_TOUCHE -> SWR2C2
- SW9: value SW_TOUCHE -> SWR2C3
